File: TCD1304Rev2KiCAD/TCD1304Rev2.kicad_pcb (KiCad board)
At the start: 4 copper layers, 60 x 40 mm, 26 parts, among them J1 Conn_01x08_Male, J2 Conn_01x16_Male, U1 TCD1304AP, U2 ADA4807-2ARMZ-R7, U3 Teensy4.0

Commit message: updated pcb
Parts:
- removed D1, D2, D3, D4, D5, D6: D_Schottky, Diode_SMD:D_SOD-323
- removed J1: Conn_01x08_Male, Connector_PinHeader_2.54mm:PinHeader_1x08_P2.54mm_Vertical
- removed R7: 300R, Resistor_SMD:R_0603_1608Metric
- added J3: Conn_01x16_Male, Connector_PinHeader_2.54mm:PinHeader_1x16_P2.54mm_Vertical, F.Cu at (139.0, 117.5)
- added REF**: MountingHole_3.2mm_M3_DIN965_Pad, MountingHole:MountingHole_3.2mm_M3_DIN965_Pad, F.Cu at (185.5, 115.5)
- added REF**: MountingHole_3.2mm_M3_DIN965_Pad, MountingHole:MountingHole_3.2mm_M3_DIN965_Pad, F.Cu at (185.5, 84.5)
- added REF**: MountingHole_3.2mm_M3_DIN965_Pad, MountingHole:MountingHole_3.2mm_M3_DIN965_Pad, F.Cu at (124.5, 84.5)
- added REF**: MountingHole_3.2mm_M3_DIN965_Pad, MountingHole:MountingHole_3.2mm_M3_DIN965_Pad, F.Cu at (124.5, 115.5)
- C1, C2, C3, C4, C5, C6, C7: footprint Capacitor_SMD:C_0603_1608Metric -> Capacitor_SMD:C_0805_2012Metric_Pad1.18x1.45mm_HandSolder
- R1, R2, R3, R4: footprint Resistor_SMD:R_0603_1608Metric -> Resistor_SMD:R_0805_2012Metric_Pad1.20x1.40mm_HandSolder
- R5, R6: value 300R -> 2.49K; footprint Resistor_SMD:R_0603_1608Metric -> Resistor_SMD:R_0805_2012Metric_Pad1.20x1.40mm_HandSolder
- moved C1 49.5 mm to (183.2, 110.5), turned to 0 degrees
- moved C6 33.3 mm to (145.8, 92.5), turned to 180 degrees
- moved C7 10.8 mm to (157.8, 110.8), turned to 0 degrees
- moved U1 9.57 mm to (159.6, 100.0)
- moved U3 9.57 mm to (170.6, 100.0)
- moved R4 5.12 mm to (139.0, 107.4)
- moved R1 3.97 mm to (141.3, 101.4)
- moved R5 3.78 mm to (169.2, 112.5), turned to -90 degrees
- moved C3 3.24 mm to (131.8, 108.4)
- moved C4 3.15 mm to (131.8, 106.4)
- moved RV1 2.79 mm to (132.0, 93.1)
- moved U2 2.79 mm to (134.5, 101.7)
- moved R2 2.54 mm to (134.5, 97.2)
- moved R6 2.30 mm to (166.8, 112.5), turned to -90 degrees
- moved R3 2.10 mm to (126.5, 102.4)
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Connections:
- R5 pad 1: Net-(J1-Pin_3) -> Net-(J3-Pin_6)
- R5 pad 2: Net-(D5-A) -> +3.3V
- R6 pad 1: Net-(J1-Pin_5) -> Net-(J3-Pin_4)
- R6 pad 2: Net-(D3-A) -> +3.3V
- U3 pad 23: Net-(D3-A) -> Net-(J3-Pin_2)
- U3 pad 24: Net-(D5-A) -> Net-(J3-Pin_3)
- U3 pad 25: unconnected-(U3-18_A4_SDA0-Pad25) -> Net-(J3-Pin_4)
- U3 pad 26: unconnected-(U3-19_A5_SCL0-Pad26) -> Net-(J3-Pin_6)
- U3 pad 27: unconnected-(U3-20_A6_TX5_LRCLK1-Pad27) -> Net-(J3-Pin_8)
- U3 pad 28: unconnected-(U3-21_A7_RX5_BCLK1-Pad28) -> Net-(J3-Pin_9)
- U3 pad 29: unconnected-(U3-22_A8_CTX1-Pad29) -> Net-(J3-Pin_10)
- U3 pad 30: unconnected-(U3-23_A9_CRX1_MCLK1-Pad30) -> Net-(J3-Pin_11)
- U3 pad 33: unconnected-(U3-VIN-Pad33) -> Net-(J3-Pin_16)
Routing:
- net Net-(J3-Pin_4): track 0.00 -> 28.1 mm
- net Net-(D5-A): track 25.6 -> 0.00 mm
- net Net-(J3-Pin_3): track 0.00 -> 24.5 mm
- net Net-(J3-Pin_2): track 0.00 -> 24.3 mm
- net Net-(J3-Pin_6): track 0.00 -> 24.0 mm
- net Net-(D3-A): track 19.2 -> 0.00 mm
- net Net-(J3-Pin_8): track 0.00 -> 19.2 mm
- net Net-(J3-Pin_11): track 0.00 -> 19.2 mm
- net Net-(J3-Pin_9): track 0.00 -> 19.2 mm
- net Net-(J3-Pin_10): track 0.00 -> 19.2 mm
- net Net-(J3-Pin_16): track 0.00 -> 14.1 mm
- net Net-(J3-Pin_1): track 14.1 -> 24.3 mm
- net Net-(J1-Pin_3): track 7.45 -> 0.00 mm
- net Net-(J2-Pin_6): track 41.0 -> 34.2 mm
- net +3.3V: track 14.7 -> 19.9 mm, vias 3 -> 4
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Other:
- board size 60 x 40 mm -> 70 x 40 mm
- board text removed: "3.3V"
- board text removed: "A1"
- board text removed: "A2"
- board text removed: "A3"
- board text removed: "GND"
- board text removed: "TCD1304 Rev2b Mitchell C Nelson, PhD Dec 26, 2024"
