File: TCD1304Rev2KiCAD/TCD1304Rev2.kicad_sch (KiCad schematic)
At the start: 26 parts, among them J1 Conn_01x08_Male, J2 Conn_01x16_Male, U1 TCD1304AP, U2 ADA4807-2ARMZ-R7, U3 Teensy4.0

Commit message: updated pcb
Parts:
- removed D1, D2, D3, D4, D5, D6: D_Schottky, Diode_SMD:D_SOD-323, symbol Device:D_Schottky
- removed J1: Conn_01x08_Male, Connector_PinHeader_2.54mm:PinHeader_1x08_P2.54mm_Vertical, symbol Connector:Conn_01x08_Male
- removed R7: 300R, Resistor_SMD:R_0603_1608Metric, symbol Device:R
- added J3: Conn_01x16_Male, Connector_PinHeader_2.54mm:PinHeader_1x16_P2.54mm_Vertical, symbol Connector:Conn_01x16_Male
- C1, C2, C3, C4, C5, C6, C7: footprint Capacitor_SMD:C_0603_1608Metric -> Capacitor_SMD:C_0805_2012Metric_Pad1.18x1.45mm_HandSolder
- R1, R2, R3, R4: footprint Resistor_SMD:R_0603_1608Metric -> Resistor_SMD:R_0805_2012Metric_Pad1.20x1.40mm_HandSolder
- R5, R6: value 300R -> 2.49K; footprint Resistor_SMD:R_0603_1608Metric -> Resistor_SMD:R_0805_2012Metric_Pad1.20x1.40mm_HandSolder; Digikey 2019-RK73H1JTTD3000FCT-ND -> 311-2.49KHRCT-ND; now not fitted
Connections:
- net +3.3V: now also R5.2, R6.2
- net Earth: now also U3.47 (GND), J3.15 (Pin_15), J3.5 (Pin_5), J3.7 (Pin_7)
- net at U3.22 (15_A1_RX3_SPDIF_IN): now also J3.1 (Pin_1)
- net at U3.24 (17_A3_TX4_SDA1): now also J3.3 (Pin_3); no longer R5.2
- net at R5.1: now also U3.26 (19_A5_SCL0), J3.6 (Pin_6)
- net at R6.1: now also U3.25 (18_A4_SDA0), J3.4 (Pin_4)
- net at U3.23 (16_A2_RX4_SCL1): now also J3.2 (Pin_2); no longer R6.2
- net at U3.27 (20_A6_TX5_LRCLK1): now also J3.8 (Pin_8)
- net at U3.28 (21_A7_RX5_BCLK1): now also J3.9 (Pin_9)
- net at U3.29 (22_A8_CTX1): now also J3.10 (Pin_10)
- net at U3.30 (23_A9_CRX1_MCLK1): now also J3.11 (Pin_11)
- net at U3.33 (VIN): now also J3.16 (Pin_16)
- no-connect marks 0 -> 28
Other:
- moved on the sheet: U3
